File: Hardware/PCB/Jarvis_v1.kicad_sch (KiCad schematic)
At the start: 28 parts, among them J1 USB_C_Power, J10 J_RFID, J2 Lipo_Connector, J3 J_ESP32_L, J4 J_ESP32_R, J5 ESP_CAM_L, J6 ESP_CAM_R, J7 Programmer, J8 J_OLED, J9 J_MIC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

Commit message: pcbupdate
Parts:
- D1, D2, D3: footprint (none) -> LED_THT:LED_D3.0mm
- J1: footprint (none) -> Connector_USB:USB_C_Receptacle_GCT_USB4125-xx-x_6P_TopMnt_Horizontal
- J10, J5, J6: footprint (none) -> Connector_PinHeader_2.54mm:PinHeader_1x08_P2.54mm_Vertical
- J2: footprint (none) -> Connector_JST:JST_PH_S2B-PH-K_1x02_P2.00mm_Horizontal
- J3, J4: footprint (none) -> Connector_PinHeader_2.54mm:PinHeader_1x19_P2.54mm_Vertical
- J7, J8, U2: footprint (none) -> Connector_PinHeader_2.54mm:PinHeader_1x04_P2.54mm_Vertical
- J9, U1: footprint (none) -> Connector_PinHeader_2.54mm:PinHeader_1x06_P2.54mm_Vertical
- R1, R2, R3, R4, R5, R6, R7, R8: footprint (none) -> Resistor_THT:R_Axial_DIN0207_L6.3mm_D2.5mm_P7.62mm_Horizontal
- SW1: footprint (none) -> Connector_PinHeader_2.54mm:PinHeader_1x03_P2.54mm_Vertical
- SW2, SW3, SW4: footprint (none) -> Button_Switch_THT:SW_PUSH_6mm_H5mm
- SW5: footprint (none) -> Rotary_Encoder:RotaryEncoder_Alps_EC11E-Switch_Vertical_H20mm
Connections:
- net RFID_RST: now also J4.16 (Pin_16)
- no-connect marks 0 -> 29
